File: pcbDesigns/mcuPower/mcuPower/mcuPower.kicad_pcb (KiCad board)
At the start: 2 copper layers, 112 x 100 mm, 10 parts, among them J1 AC_IN, J2 DC_OUT_1, J3 DC_OUT_2, T1 Transformer_1P_1S_230:24

Commit message: bugfix
fix wron connecter direction
Parts:
- moved J2 5.12 mm to (143.1, 59.0), turned to 180 degrees
- moved C3 5.00 mm to (143.0, 70.0), turned to 180 degrees
Changed lines of the file:
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@@
   )
   (footprint "Capacitor_THT:C_Disc_D5.1mm_W3.2mm_P5.00mm" (layer "F.Cu")
-    (at 138 70)
+    (at 143 70 180)
     (descr "C, Disc series, Radial, pin pitch=5.00mm, , diameter*width=5.1*3.2mm^2, Capacitor, http://www.vishay.com/docs/45233/krseries.pdf")
     (tags "C Disc series Radial pin pitch 5.00mm  diameter 5.1mm width 3.2mm Capacitor")
@@
     (fp_line (start -0.05 1.6) (end 5.05 1.6) (layer "F.Fab") (width 0.1))
     (fp_line (start 5.05 1.6) (end 5.05 -1.6) (layer "F.Fab") (width 0.1))
-    (pad "1" thru_hole circle (at 0 0) (size 1.6 1.6) (drill 0.8) (layers *.Cu *.Mask)
+    (pad "1" thru_hole circle (at 0 0 180) (size 1.6 1.6) (drill 0.8) (layers *.Cu *.Mask)
       (net 1 "VCC") (pintype "passive"))
-    (pad "2" thru_hole circle (at 5 0) (size 1.6 1.6) (drill 0.8) (layers *.Cu *.Mask)
+    (pad "2" thru_hole circle (at 5 0 180) (size 1.6 1.6) (drill 0.8) (layers *.Cu *.Mask)
       (net 2 "GND") (pintype "passive"))
     (model "${KICAD6_3DMODEL_DIR}/Capacitor_THT.3dshapes/C_Disc_D5.1mm_W3.2mm_P5.00mm.wrl"
@@
   )
   (footprint "TerminalBlock_MetzConnect:TerminalBlock_MetzConnect_Type101_RT01602HBWC_1x02_P5.08mm_Horizontal" (layer "F.Cu")
-    (at 137.955 59)
+    (at 143.08 59 180)
     (descr "terminal block Metz Connect Type101_RT01602HBWC, 2 pins, pitch 5.08mm, size 10.2x8mm^2, drill diamater 1.3mm, pad diameter 2.5mm, see http://www.metz-connect.com/de/system/files/productfiles/Datenblatt_311011_RT016xxHBWC_OFF-022771S.pdf, script-generated using https://github.com/pointhi/kicad-footprint-generator/scripts/TerminalBlock_MetzConnect")
     (tags "THT terminal block Metz Connect Type101_RT01602HBWC pitch 5.08mm size 10.2x8mm^2 drill 1.3mm pad 2.5mm")
@@
     (fp_circle (center 5.08 0) (end 6.58 0) (layer "F.Fab") (width 0.1) (fill none))
     (fp_circle (center 0 0) (end 1.5 0) (layer "F.Fab") (width 0.1) (fill none))
-    (pad "1" thru_hole rect (at 0 0) (size 2.5 2.5) (drill 1.3) (layers *.Cu *.Mask)
+    (pad "1" thru_hole rect (at 0 0 180) (size 2.5 2.5) (drill 1.3) (layers *.Cu *.Mask)
       (net 1 "VCC") (pinfunction "Pin_1") (pintype "passive"))
-    (pad "2" thru_hole circle (at 5.08 0) (size 2.5 2.5) (drill 1.3) (layers *.Cu *.Mask)
+    (pad "2" thru_hole circle (at 5.08 0 180) (size 2.5 2.5) (drill 1.3) (layers *.Cu *.Mask)
       (net 2 "GND") (pinfunction "Pin_2") (pintype "passive"))
     (model "${KICAD6_3DMODEL_DIR}/TerminalBlock_MetzConnect.3dshapes/TerminalBlock_MetzConnect_Type101_RT01602HBWC_1x02_P5.08mm_Horizontal.wrl"
@@
         (xy 121 86.5)
         (xy 121 79.5)
-        (xy 121 79.5)
         (xy 121 51)
